File: sch/Memory2.sch (KiCad schematic (older format))
At the start: 31 parts

Commit message: Updated the code and circuit diagrams for first boot from banked RAM.
Parts:
- removed U? (x3): 74LS139, symbol 74LS139
- removed U? (x2): 74LS32, symbol 74LS32
- added C?: 0.1uF, symbol C
- added IC?: 74HC138, symbol 74HC138
- added IC? (x2): 74HC04, 108-5299, symbol 74HC04
- added R? (x16): 10k, symbol R
- added U?: 74LS139, symbol 74LS139
- added U?: 74LS32, symbol 74LS32
Connections:
- net A0: now also IC?.1 (A0)
- net A1: now also IC?.2 (A1)
- net A2: now also IC?.3 (A2)
- net A3: now also IC?.4 (E1)
- net BA14: now also R?.2
- net BA15: now also R?.2
- net BA16: now also R?.2
- net BA17: now also R?.2
- net BA18: now also R?.2
- net BA19: now also R?.2
- net BA20: now also R?.2
- net BA21: now also R?.2
- net B_WR0: now also IC?.15 (Y0)
- net B_WR1: now also IC?.14 (Y1)
- net B_WR2: now also IC?.13 (Y2)
- net B_WR3: now also IC?.12 (Y3)
- net D0: now also IC?.18 (B0); no longer IC?.2 (A0)
- net D1: now also IC?.17 (B1); no longer IC?.3 (A1)
- net D2: now also IC?.16 (B2); no longer IC?.4 (A2)
- net D3: now also IC?.15 (B3); no longer IC?.5 (A3)
- net D4: now also IC?.14 (B4); no longer IC?.6 (A4)
- net D5: now also IC?.13 (B5); no longer IC?.7 (A5)
- net D6: now also IC?.12 (B6); no longer IC?.8 (A6)
- net D7: now also IC?.11 (B7); no longer IC?.9 (A7)
- net GND: now also IC?.19 (CE), C?.2, IC?.7 (GND), IC?.7 (GND), IC?.8 (GND), R?.1, R?.1, R?.1, R?.1, R?.1, R?.1, R?.1, R?.1, R?.1, R?.1, R?.1, R?.1, R?.1, R?.1, R?.1, R?.1, U?.7 (GND), U?.8 (GND); no longer U?.1 (E)
- net MD0: now also IC?.2 (A0), R?.2; no longer IC?.18 (B0)
- net MD1: now also IC?.3 (A1), R?.2; no longer IC?.17 (B1)
- net MD2: now also IC?.4 (A2), R?.2; no longer IC?.16 (B2)
- net MD3: now also IC?.5 (A3), R?.2; no longer IC?.15 (B3)
- net MD4: now also IC?.6 (A4), R?.2; no longer IC?.14 (B4)
- net MD5: now also IC?.7 (A5), R?.2; no longer IC?.13 (B5)
- net MD6: now also IC?.8 (A6), R?.2; no longer IC?.12 (B6)
- net MD7: now also IC?.9 (A7), R?.2; no longer IC?.11 (B7)
- net MEM_CFG: now also IC?.1
- net MREQ: now also U?.2; no longer IC?.19 (CE)
- net RD: now also U?.1; no longer IC?.1 (A->B)
- net VCC: now also IC?.14 (VCC), IC?.14 (VCC), U?.14 (VCC), U?.16 (VCC)
- net WR: now also IC?.5 (E2)
- net at U?.11 (Cp): now also IC?.11 (Y4)
- net at IC?.2: now also U?.1 (E)
- new net: IC?.1 (A->B), IC?.2
- new net: IC?.2, IC?.6 (E3)
- new net: IC?.1, U?.3
- new net +5V: C?.1, IC?.16 (Vcc), U?.1 (E)
- no-connect marks 12 -> 16
