File: sch/iodecode.sch (KiCad schematic (older format))
At the start: 3 parts

Commit message: Added new schematics and about to start coding for new MMU.
Connections:
- net MEM_CFG: now reaches IC?.3 (Y2)
- no-connect marks 29 -> 28
Changed lines of the file:
@@
-EESchema Schematic File Version 2  date Fri 17 Dec 2010 20:03:20 GMT
+EESchema Schematic File Version 2  date Sat 19 Feb 2011 16:33:30 GMT
 LIBS:74xx
 LIBS:adc-dac
@@
 EELAYER END
 $Descr A4 11700 8267
-Sheet 5 12
+Sheet 9 13
 Title ""
-Date "17 dec 2010"
+Date "19 feb 2011"
 Rev ""
 Comp ""
@@
 Comment4 ""
 $EndDescr
+Wire Wire Line
+	4500 2400 4600 2400
+Wire Wire Line
+	7800 4200 7900 4200
+Wire Wire Line
+	7800 4100 7900 4100
+Wire Wire Line
+	7800 4000 7900 4000
+Wire Wire Line
+	7800 3900 7900 3900
+Wire Wire Line
+	7800 3800 7900 3800
+Wire Wire Line
+	7800 3700 7900 3700
+Wire Wire Line
+	7800 3600 7900 3600
+Wire Wire Line
+	7800 3500 7900 3500
+Wire Wire Line
+	7800 2400 7900 2400
+Wire Wire Line
+	7800 2300 7900 2300
+Wire Wire Line
+	7800 2200 7900 2200
+Wire Wire Line
+	7800 2100 7900 2100
+Wire Wire Line
+	7800 2000 7900 2000
+Wire Wire Line
+	7800 1900 7900 1900
+Wire Wire Line
+	7800 1800 7900 1800
+Wire Wire Line
+	7800 1700 7900 1700
+Wire Wire Line
+	6100 3300 6100 3200
+Wire Wire Line
+	6100 3200 6200 3200
+Wire Wire Line
+	6200 4900 6100 4900
+Connection ~ 5750 2000
+Wire Wire Line
+	5350 2000 6200 2000
+Connection ~ 5550 1800
+Wire Wire Line
+	5350 1800 6200 1800
+Wire Wire Line
+	5450 1700 5450 3500
+Wire Wire Line
+	5450 3500 6200 3500
+Wire Wire Line
+	5650 1900 5650 3700
+Wire Wire Line
+	5650 3700 6200 3700
+Connection ~ 5850 2200
+Wire Wire Line
+	5850 2200 5850 4000
+Wire Wire Line
+	5850 4000 6200 4000
+Wire Wire Line
+	6200 2300 6100 2300
+Wire Wire Line
+	2900 2500 2800 2500
+Wire Wire Line
+	2900 2400 2800 2400
+Wire Wire Line
+	2900 2300 2800 2300
+Wire Wire Line
+	2900 2200 2800 2200
+Wire Wire Line
+	2800 3800 2800 3700
+Wire Wire Line
+	2800 3700 2900 3700
+Wire Wire Line
+	2800 2700 2900 2700
+Wire Wire Line
+	2900 2800 2800 2800
+Wire Wire Line
+	2800 2800 2800 2900
+Wire Wire Line
+	2900 3600 2800 3600
+Wire Wire Line
+	2800 3600 2800 3500
+Wire Wire Line
+	4500 2200 6200 2200
+Wire Wire Line
+	6100 4100 6200 4100
+Wire Wire Line
+	5750 2000 5750 3800
+Wire Wire Line
+	5750 3800 6200 3800
+Wire Wire Line
+	5550 1800 5550 3600
+Wire Wire Line
+	5550 3600 6200 3600
+Wire Wire Line
+	5350 1700 6200 1700
+Connection ~ 5450 1700
+Wire Wire Line
+	5350 1900 6200 1900
+Connection ~ 5650 1900
+Wire Wire Line
+	6100 4900 6100 4800
+Wire Wire Line
+	6200 5000 6100 5000
+Wire Wire Line
+	6100 5000 6100 5100
+Wire Wire Line
+	6200 3100 6100 3100
+Wire Wire Line
+	6100 3100 6100 3000
+Wire Wire Line
+	7800 2500 7900 2500
+Wire Wire Line
+	4500 2300 4600 2300
+Text GLabel 4600 2400 2    60   Output ~ 0
+MEM_CFG
 NoConn ~ 4500 3700
 NoConn ~ 4500 3600
@@
 NoConn ~ 4500 2600
 NoConn ~ 4500 2500
-NoConn ~ 4500 2400
-Wire Wire Line
-	4500 2300 4600 2300
-Wire Wire Line
-	7800 2500 7900 2500
-Wire Wire Line
-	6100 3000 6100 3100
-Wire Wire Line
-	6100 3100 6200 3100
-Wire Wire Line
-	6100 5100 6100 5000
-Wire Wire Line
-	6100 5000 6200 5000
-Wire Wire Line
-	6100 4800 6100 4900
-Connection ~ 5650 1900
-Wire Wire Line
-	5350 1900 6200 1900
-Connection ~ 5450 1700
-Wire Wire Line
-	5350 1700 6200 1700
-Wire Wire Line
-	6200 3600 5550 3600
-Wire Wire Line
-	5550 3600 5550 1800
-Wire Wire Line
-	6200 3800 5750 3800
-Wire Wire Line
-	5750 3800 5750 2000
-Wire Wire Line
-	6100 4100 6200 4100
-Wire Wire Line
-	4500 2200 6200 2200
-Wire Wire Line
-	2800 3500 2800 3600
-Wire Wire Line
-	2800 3600 2900 3600
-Wire Wire Line
-	2800 2900 2800 2800
-Wire Wire Line
-	2800 2800 2900 2800
-Wire Wire Line
-	2800 2700 2900 2700
-Wire Wire Line
-	2900 3700 2800 3700
-Wire Wire Line
-	2800 3700 2800 3800
-Wire Wire Line
-	2900 2200 2800 2200
-Wire Wire Line
-	2900 2300 2800 2300
-Wire Wire Line
-	2900 2400 2800 2400
-Wire Wire Line
-	2900 2500 2800 2500
-Wire Wire Line
-	6200 2300 6100 2300
-Wire Wire Line
-	6200 4000 5850 4000
-Wire Wire Line
-	5850 4000 5850 2200
-Connection ~ 5850 2200
-Wire Wire Line
-	6200 3700 5650 3700
-Wire Wire Line
-	5650 3700 5650 1900
-Wire Wire Line
-	6200 3500 5450 3500
-Wire Wire Line
-	5450 3500 5450 1700
-Wire Wire Line
-	5350 1800 6200 1800
-Connection ~ 5550 1800
-Wire Wire Line
-	5350 2000 6200 2000
-Connection ~ 5750 2000
-Wire Wire Line
-	6100 4900 6200 4900
-Wire Wire Line
-	6200 3200 6100 3200
-Wire Wire Line
-	6100 3200 6100 3300
-Wire Wire Line
-	7800 1700 7900 1700
-Wire Wire Line
-	7800 1800 7900 1800
-Wire Wire Line
-	7800 1900 7900 1900
-Wire Wire Line
-	7800 2000 7900 2000
-Wire Wire Line
-	7800 2100 7900 2100
-Wire Wire Line
-	7800 2200 7900 2200
-Wire Wire Line
-	7800 2300 7900 2300
-Wire Wire Line
-	7800 2400 7900 2400
-Wire Wire Line
-	7800 3500 7900 3500
-Wire Wire Line
-	7800 3600 7900 3600
-Wire Wire Line
-	7800 3700 7900 3700
-Wire Wire Line
-	7800 3800 7900 3800
-Wire Wire Line
-	7800 3900 7900 3900
-Wire Wire Line
-	7800 4000 7900 4000
-Wire Wire Line
-	7800 4100 7900 4100
-Wire Wire Line
-	7800 4200 7900 4200
 Text GLabel 4600 2300 2    60   Output ~ 0
 CLK_CS
