File: sch/keyboard.sch (KiCad schematic (older format))
At the start: 19 parts, among them IC13 PIC18F4520-DIP, IC20 74HC08

Commit message: Updated the code and circuit diagrams for first boot from banked RAM.
Parts:
- added JP?: JUMPER, symbol JUMPER
Connections:
- net at IC13.1 (#MCLR/Vpp/RE3), R?.1: now also JP?.1
- new net Z80_RST: JP?.2
Changed lines of the file:
@@
-EESchema Schematic File Version 2  date Sat 19 Feb 2011 16:33:30 GMT
+EESchema Schematic File Version 2  date Sun 06 Mar 2011 19:20:09 GMT
 LIBS:74xx
 LIBS:adc-dac
@@
 EELAYER END
 $Descr A4 11700 8267
-Sheet 3 13
+Sheet 7 13
 Title ""
-Date "19 feb 2011"
+Date "6 mar 2011"
 Rev ""
 Comp ""
@@
 Comment4 ""
 $EndDescr
+Text GLabel 6650 5350 2    60   Input ~ 0
+Z80_RST
+Wire Wire Line
+	6200 5350 6650 5350
 Connection ~ 4100 1800
 Connection ~ 4000 4250
 Wire Wire Line
-	4000 1800 4000 4250
+	4000 4250 4000 1800
 Wire Wire Line
 	4000 1800 4300 1800
@@
 Wire Wire Line
 	4300 1800 4300 1900
+Wire Wire Line
+	5600 5150 5600 5350
+Wire Wire Line
+	5600 5350 5800 5350
+Connection ~ 5600 5150
+$Comp
+L JUMPER JP?
+U 1 1 4D73DBE5
+P 6000 5350
+F 0 "JP?" H 6000 5500 60  0000 C CNN
+F 1 "JUMPER" H 6000 5270 40  0000 C CNN
+	1    6000 5350
+	1    0    0    -1
+$EndComp
 $Comp
 L GND #PWR?
